File: Mult/Mult.kicad_sch (KiCad schematic)
At the start: 5 parts, among them J1 IN, J2 OUT1, J3 OUT2, J4 OUT3, J5 OUT4

Commit message: add footprint model
Parts:
- J1, J2, J3, J4: footprint Connector_Audio:Jack_3.5mm_QingPu_WQP-PJ398SM_Vertical_CircularHoles -> pj398m:Jack_3.5mm_QingPu_WQP-PJ398SM_Vertical
- J5: footprint (none) -> pj398m:Jack_3.5mm_QingPu_WQP-PJ398SM_Vertical
Changed lines of the file:
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@@
       (effects (font (size 1.27 1.27)) (justify right))
     )
-    (property "Footprint" "Connector_Audio:Jack_3.5mm_QingPu_WQP-PJ398SM_Vertical_CircularHoles" (id 2) (at 140.97 104.14 0)
+    (property "Footprint" "pj398m:Jack_3.5mm_QingPu_WQP-PJ398SM_Vertical" (id 2) (at 140.97 104.14 0)
       (effects (font (size 1.27 1.27)) hide)
     )
@@
       (effects (font (size 1.27 1.27)) (justify right))
     )
-    (property "Footprint" "" (id 2) (at 140.97 120.65 0)
+    (property "Footprint" "pj398m:Jack_3.5mm_QingPu_WQP-PJ398SM_Vertical" (id 2) (at 140.97 120.65 0)
       (effects (font (size 1.27 1.27)) hide)
     )
@@
       (effects (font (size 1.27 1.27)) (justify right))
     )
-    (property "Footprint" "Connector_Audio:Jack_3.5mm_QingPu_WQP-PJ398SM_Vertical_CircularHoles" (id 2) (at 140.97 68.58 0)
+    (property "Footprint" "pj398m:Jack_3.5mm_QingPu_WQP-PJ398SM_Vertical" (id 2) (at 140.97 68.58 0)
       (effects (font (size 1.27 1.27)) hide)
     )
@@
     (property "Reference" "J1" (id 0) (at 103.505 86.36 0))
     (property "Value" "IN" (id 1) (at 103.505 88.9 0))
-    (property "Footprint" "Connector_Audio:Jack_3.5mm_QingPu_WQP-PJ398SM_Vertical_CircularHoles" (id 2) (at 104.14 95.25 0)
+    (property "Footprint" "pj398m:Jack_3.5mm_QingPu_WQP-PJ398SM_Vertical" (id 2) (at 104.14 95.25 0)
       (effects (font (size 1.27 1.27)) hide)
     )
@@
       (effects (font (size 1.27 1.27)) (justify right))
     )
-    (property "Footprint" "Connector_Audio:Jack_3.5mm_QingPu_WQP-PJ398SM_Vertical_CircularHoles" (id 2) (at 140.97 86.36 0)
+    (property "Footprint" "pj398m:Jack_3.5mm_QingPu_WQP-PJ398SM_Vertical" (id 2) (at 140.97 86.36 0)
       (effects (font (size 1.27 1.27)) hide)
     )
@@
     )
     (path "/9a9a7b80-7913-41bb-b84f-4f70c87fac29"
-      (reference "J1") (unit 1) (value "IN") (footprint "Connector_Audio:Jack_3.5mm_QingPu_WQP-PJ398SM_Vertical_CircularHoles")
+      (reference "J1") (unit 1) (value "IN") (footprint "pj398m:Jack_3.5mm_QingPu_WQP-PJ398SM_Vertical")
     )
     (path "/2ef1383a-a610-42dc-8dd9-459d5c00acc9"
-      (reference "J2") (unit 1) (value "OUT1") (footprint "Connector_Audio:Jack_3.5mm_QingPu_WQP-PJ398SM_Vertical_CircularHoles")
+      (reference "J2") (unit 1) (value "OUT1") (footprint "pj398m:Jack_3.5mm_QingPu_WQP-PJ398SM_Vertical")
     )
     (path "/fd29545e-e8bf-4f59-9531-5a642f9144b3"
-      (reference "J3") (unit 1) (value "OUT2") (footprint "Connector_Audio:Jack_3.5mm_QingPu_WQP-PJ398SM_Vertical_CircularHoles")
+      (reference "J3") (unit 1) (value "OUT2") (footprint "pj398m:Jack_3.5mm_QingPu_WQP-PJ398SM_Vertical")
     )
     (path "/19f91c85-22f0-48ec-9e7d-6d551482c991"
-      (reference "J4") (unit 1) (value "OUT3") (footprint "Connector_Audio:Jack_3.5mm_QingPu_WQP-PJ398SM_Vertical_CircularHoles")
+      (reference "J4") (unit 1) (value "OUT3") (footprint "pj398m:Jack_3.5mm_QingPu_WQP-PJ398SM_Vertical")
     )
     (path "/2de0684d-1228-40f9-83f6-95302c40bb30"
-      (reference "J5") (unit 1) (value "OUT4") (footprint "Connector_Audio:Jack_3.5mm_QingPu_WQP-PJ398SM_Vertical_CircularHoles")
+      (reference "J5") (unit 1) (value "OUT4") (footprint "pj398m:Jack_3.5mm_QingPu_WQP-PJ398SM_Vertical")
     )
   )
