File: ASREnvelope/ASREnvelope.kicad_sch (KiCad schematic)
At the start: 45 parts

Commit message: rearrange a bunch of files
Parts:
- C1, C8: value (none) -> 1uF; footprint (none) -> Capacitor_THT:C_Disc_D3.0mm_W1.6mm_P2.50mm
- C2, C3: value (none) -> 10uF; footprint (none) -> Capacitor_THT:CP_Radial_D5.0mm_P2.50mm
- C4, C5, C6, C7: value (none) -> 0.1uF; footprint (none) -> Capacitor_THT:C_Disc_D11.0mm_W5.0mm_P7.50mm
- D1, D4, D5, D6, D7, D8: value (none) -> 1N4148; footprint (none) -> Diode_THT:D_DO-35_SOD27_P7.62mm_Horizontal
- D2, D3: value (none) -> 1N5819; footprint (none) -> Diode_THT:D_DO-41_SOD81_P7.62mm_Horizontal
- J1: value (none) -> GATE; footprint (none) -> pj398m:Jack_3.5mm_QingPu_WQP-PJ398SM_Vertical
- J2: value (none) -> Power; footprint (none) -> pj398m:Jack_3.5mm_QingPu_WQP-PJ398SM_Vertical
- J3: value (none) -> OUT; footprint (none) -> pj398m:Jack_3.5mm_QingPu_WQP-PJ398SM_Vertical
- J4: value (none) -> INV OUT; footprint (none) -> pj398m:Jack_3.5mm_QingPu_WQP-PJ398SM_Vertical
- J5: value (none) -> Conn_01x06_Male; footprint (none) -> Connector_PinHeader_2.54mm:PinHeader_1x06_P2.54mm_Vertical
- J6: value (none) -> Conn_01x04_Male; footprint (none) -> Connector_PinHeader_2.54mm:PinHeader_1x04_P2.54mm_Vertical
- J7: value (none) -> Conn_01x04_Female; footprint (none) -> Connector_PinSocket_2.54mm:PinSocket_1x04_P2.54mm_Vertical
- J8: value (none) -> Conn_01x06_Female; footprint (none) -> Connector_PinSocket_2.54mm:PinSocket_1x06_P2.54mm_Vertical
- R1: value (none) -> 10K; footprint (none) -> Resistor_THT:R_Axial_DIN0207_L6.3mm_D2.5mm_P7.62mm_Horizontal
- R10, R11, R12, R13, R2, R4, R5, R6, R7, R9: value (none) -> 100K; footprint (none) -> Resistor_THT:R_Axial_DIN0207_L6.3mm_D2.5mm_P7.62mm_Horizontal
- R14, R15: value (none) -> 1K; footprint (none) -> Resistor_THT:R_Axial_DIN0207_L6.3mm_D2.5mm_P7.62mm_Horizontal
- R3: value (none) -> 47K; footprint (none) -> Resistor_THT:R_Axial_DIN0207_L6.3mm_D2.5mm_P7.62mm_Horizontal
- R8: value (none) -> 100; footprint (none) -> Resistor_THT:R_Axial_DIN0207_L6.3mm_D2.5mm_P7.62mm_Horizontal
- RV1: value (none) -> A100K Sustain; footprint (none) -> Potentiometer_THT:Potentiometer_Alpha_RD901F-40-00D_Single_Vertical_CircularHoles
- RV2: value (none) -> A1M Attack; footprint (none) -> Potentiometer_THT:Potentiometer_Alpha_RD901F-40-00D_Single_Vertical_CircularHoles
- RV3: value (none) -> A1M Decay/Release; footprint (none) -> Potentiometer_THT:Potentiometer_Alpha_RD901F-40-00D_Single_Vertical_CircularHoles
- SW1: value (none) -> SW_SPDT
- U1: value (none) -> TL074; footprint (none) -> Package_DIP:DIP-16_W7.62mm_Socket_LongPads
- U2: value (none) -> TL072; footprint (none) -> Package_DIP:DIP-8_W7.62mm_Socket_LongPads

Commit message: add eurocad footprint library
Parts:
- J2: footprint pj398m:Jack_3.5mm_QingPu_WQP-PJ398SM_Vertical -> Connector_PinHeader_2.54mm:PinHeader_2x05_P2.54mm_Horizontal
- RV1, RV2, RV3: footprint Potentiometer_THT:Potentiometer_Alpha_RD901F-40-00D_Single_Vertical_CircularHoles -> Eurocad:Alpha9mmPot
- SW1: footprint (none) -> Eurocad:SPDT toggle on-off-on
Changed lines of the file:
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@@
     (property "Reference" "J2" (id 0) (at 58.42 165.9382 0))
     (property "Value" "Power" (id 1) (at 58.42 168.2496 0))
-    (property "Footprint" "pj398m:Jack_3.5mm_QingPu_WQP-PJ398SM_Vertical" (id 2) (at 57.15 176.53 0)
+    (property "Footprint" "Connector_PinHeader_2.54mm:PinHeader_2x05_P2.54mm_Horizontal" (id 2) (at 57.15 176.53 0)
       (effects (font (size 1.27 1.27)) hide)
     )
@@
     (property "Reference" "RV1" (id 0) (at 86.36 101.981 90))
     (property "Value" "A100K Sustain" (id 1) (at 86.36 104.2924 90))
-    (property "Footprint" "Potentiometer_THT:Potentiometer_Alpha_RD901F-40-00D_Single_Vertical_CircularHoles" (id 2) (at 86.36 99.06 0)
+    (property "Footprint" "Eurocad:Alpha9mmPot" (id 2) (at 86.36 99.06 0)
       (effects (font (size 1.27 1.27)) hide)
     )
@@
     (property "Reference" "SW1" (id 0) (at 121.92 99.695 0))
     (property "Value" "SW_SPDT" (id 1) (at 121.92 102.0064 0))
-    (property "Footprint" "" (id 2) (at 121.92 107.95 0)
+    (property "Footprint" "Eurocad:SPDT toggle on-off-on" (id 2) (at 121.92 107.95 0)
       (effects (font (size 1.27 1.27)) hide)
     )
@@
     (property "Reference" "RV2" (id 0) (at 109.22 126.8222 90))
     (property "Value" "A1M Attack" (id 1) (at 109.22 129.1336 90))
-    (property "Footprint" "Potentiometer_THT:Potentiometer_Alpha_RD901F-40-00D_Single_Vertical_CircularHoles" (id 2) (at 109.22 132.08 0)
+    (property "Footprint" "Eurocad:Alpha9mmPot" (id 2) (at 109.22 132.08 0)
       (effects (font (size 1.27 1.27)) hide)
     )
@@
     (property "Reference" "RV3" (id 0) (at 109.22 148.971 90))
     (property "Value" "A1M Decay/Release" (id 1) (at 109.22 151.2824 90))
-    (property "Footprint" "Potentiometer_THT:Potentiometer_Alpha_RD901F-40-00D_Single_Vertical_CircularHoles" (id 2) (at 109.22 146.05 0)
+    (property "Footprint" "Eurocad:Alpha9mmPot" (id 2) (at 109.22 146.05 0)
       (effects (font (size 1.27 1.27)) hide)
     )
@@
     )
     (path "/00000000-0000-0000-0000-000062d57778"
-      (reference "J2") (unit 1) (value "Power") (footprint "pj398m:Jack_3.5mm_QingPu_WQP-PJ398SM_Vertical")
+      (reference "J2") (unit 1) (value "Power") (footprint "Connector_PinHeader_2.54mm:PinHeader_2x05_P2.54mm_Horizontal")
     )
     (path "/00000000-0000-0000-0000-000062cc766f"
@@
     )
     (path "/00000000-0000-0000-0000-000062d871a1"
-      (reference "RV1") (unit 1) (value "A100K Sustain") (footprint "Potentiometer_THT:Potentiometer_Alpha_RD901F-40-00D_Single_Vertical_CircularHoles")
+      (reference "RV1") (unit 1) (value "A100K Sustain") (footprint "Eurocad:Alpha9mmPot")
     )
     (path "/00000000-0000-0000-0000-000062daef05"
-      (reference "RV2") (unit 1) (value "A1M Attack") (footprint "Potentiometer_THT:Potentiometer_Alpha_RD901F-40-00D_Single_Vertical_CircularHoles")
+      (reference "RV2") (unit 1) (value "A1M Attack") (footprint "Eurocad:Alpha9mmPot")
     )
     (path "/00000000-0000-0000-0000-000062db3cbe"
-      (reference "RV3") (unit 1) (value "A1M Decay/Release") (footprint "Potentiometer_THT:Potentiometer_Alpha_RD901F-40-00D_Single_Vertical_CircularHoles")
+      (reference "RV3") (unit 1) (value "A1M Decay/Release") (footprint "Eurocad:Alpha9mmPot")
     )
     (path "/00000000-0000-0000-0000-000062d96159"
-      (reference "SW1") (unit 1) (value "SW_SPDT") (footprint "")
+      (reference "SW1") (unit 1) (value "SW_SPDT") (footprint "Eurocad:SPDT toggle on-off-on")
     )
     (path "/00000000-0000-0000-0000-000062d53133"
