File: ASREnvelope/ASREnvelope_power/ASREnvelope_power.kicad_sch (KiCad schematic)
At the start: 26 parts, among them J2 Power, J7 Conn_01x04_Female, J8 Conn_01x06_Female, U1 TL074, U2 TL072

Commit message: work on power traces
Connections:
- net +12V: now also D3.2 (A), J2.10 (Pin_10), J2.9 (Pin_9), U2.8 (V+); no longer U2.4 (V-)
- net -12V: now also D2.1 (K), J2.1 (Pin_1), J2.2 (Pin_2), U2.4 (V-); no longer U2.8 (V+)
- net Conn1B: now also J7.2 (Pin_2); no longer J7.1 (Pin_1)
- net Conn3B: now also C8.1, J8.2 (Pin_2), U2.3 (+); no longer J7.3 (Pin_3), U1.8, U1.9 (-)
- net GND: now also J8.5 (Pin_5), R3.1; no longer J7.2 (Pin_2)
- net GateJackB: now also J7.1 (Pin_1); no longer J8.1 (Pin_1)
- net InvOutJackB': now also J8.4 (Pin_4); no longer J8.3 (Pin_3)
- net OutJackB: now also J8.3 (Pin_3); no longer J8.2 (Pin_2)
- net Switch1B: now also J8.1 (Pin_1); no longer J8.4 (Pin_4)
- net Switch2B: now also J7.4 (Pin_4); no longer J8.5 (Pin_5)
- removed net Conn4B: C8.1, J7.4 (Pin_4), U2.3 (+)
- new net Conn2B: J7.3 (Pin_3), U1.8, U1.9 (-)
Other:
- moved on the sheet: U2C

Commit message: finish traces
Connections:
- net +12V: no longer C3.1, C5.2, C7.2, D3.1 (K), R10.1, R2.2, R9.2, U1.4 (V+), U2.8 (V+)
- net -12V: no longer C2.2, C4.1, C6.1, D2.2 (A), U1.11 (V-), U2.4 (V-)
- new net +12: C3.1, C5.2, C7.2, D3.1 (K), R10.1, R2.2, R9.2, U1.4 (V+), U2.8 (V+)
- new net -12: C2.2, C4.1, C6.1, D2.2 (A), U1.11 (V-), U2.4 (V-)
Changed lines of the file:
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@@
     )
   )
-  (global_label "+12V" (shape input) (at 55.88 40.64 180) (fields_autoplaced)
+  (global_label "+12" (shape input) (at 55.88 40.64 180) (fields_autoplaced)
     (effects (font (size 1.27 1.27)) (justify right))
-    (property "Intersheet References" "${INTERSHEET_REFS}" (id 0) (at 0 0 0)
-      (effects (font (size 1.27 1.27)) hide)
+    (property "Intersheet References" "${INTERSHEET_REFS}" (id 0) (at 49.4755 40.5606 0)
+      (effects (font (size 1.27 1.27)) (justify right) hide)
     )
   )
@@
     )
   )
-  (global_label "+12V" (shape input) (at 170.18 59.69 0) (fields_autoplaced)
+  (global_label "+12" (shape input) (at 170.18 59.69 0) (fields_autoplaced)
     (effects (font (size 1.27 1.27)) (justify left))
-    (property "Intersheet References" "${INTERSHEET_REFS}" (id 0) (at 0 0 0)
-      (effects (font (size 1.27 1.27)) hide)
+    (property "Intersheet References" "${INTERSHEET_REFS}" (id 0) (at 176.5845 59.6106 0)
+      (effects (font (size 1.27 1.27)) (justify left) hide)
     )
   )
@@
     )
   )
-  (global_label "+12V" (shape input) (at 231.14 74.93 180) (fields_autoplaced)
+  (global_label "+12" (shape input) (at 231.14 74.93 180) (fields_autoplaced)
     (effects (font (size 1.27 1.27)) (justify right))
-    (property "Intersheet References" "${INTERSHEET_REFS}" (id 0) (at 0 0 0)
-      (effects (font (size 1.27 1.27)) hide)
+    (property "Intersheet References" "${INTERSHEET_REFS}" (id 0) (at 224.7355 74.8506 0)
+      (effects (font (size 1.27 1.27)) (justify right) hide)
     )
   )
@@
     )
   )
-  (global_label "+12V" (shape input) (at 121.92 127 0) (fields_autoplaced)
+  (global_label "+12" (shape input) (at 121.92 127 0) (fields_autoplaced)
     (effects (font (size 1.27 1.27)) (justify left))
-    (property "Intersheet References" "${INTERSHEET_REFS}" (id 0) (at 2.54 -57.15 0)
-      (effects (font (size 1.27 1.27)) hide)
+    (property "Intersheet References" "${INTERSHEET_REFS}" (id 0) (at 128.3245 126.9206 0)
+      (effects (font (size 1.27 1.27)) (justify left) hide)
     )
   )
-  (global_label "-12V" (shape input) (at 121.92 111.76 0) (fields_autoplaced)
+  (global_label "-12" (shape input) (at 121.92 111.76 0) (fields_autoplaced)
     (effects (font (size 1.27 1.27)) (justify left))
-    (property "Intersheet References" "${INTERSHEET_REFS}" (id 0) (at 2.54 -57.15 0)
-      (effects (font (size 1.27 1.27)) hide)
+    (property "Intersheet References" "${INTERSHEET_REFS}" (id 0) (at 128.3245 111.6806 0)
+      (effects (font (size 1.27 1.27)) (justify left) hide)
     )
   )
