File: ASREnvelope/ASREnvelope_power/ASREnvelope_power.kicad_pcb (KiCad board)
At the start: 2 copper layers, 26 parts, among them J2 Power, J7 Conn_01x04_Female, J8 Conn_01x06_Female, U1 TL074, U2 TL072

Commit message: work on power traces
Parts:
- moved U1 70.7 mm to (182.7, 101.7), turned to 180 degrees
- moved J8 68.2 mm to (173.2, 122.3), turned to 90 degrees
- moved J2 60.9 mm to (174.3, 59.3), turned to 90 degrees
- moved R11 57.5 mm to (170.7, 128.7)
- moved R13 56.1 mm to (175.7, 125.6)
- moved C4 56.1 mm to (173.0, 118.5), turned to 90 degrees
- moved R12 55.1 mm to (188.5, 128.7), turned to 180 degrees
- moved D3 54.9 mm to (186.9, 70.2), turned to 90 degrees
- moved U2 46.7 mm to (177.3, 110.6)
- moved R10 41.7 mm to (188.0, 107.1), turned to -90 degrees
- moved R6 38.9 mm to (171.3, 83.3), turned to -90 degrees
- moved C5 38.2 mm to (172.2, 106.2)
- moved J7 38.2 mm to (175.8, 80.0), turned to 90 degrees
- moved C7 38.0 mm to (175.8, 69.6)
- moved C3 36.7 mm to (183.6, 63.9), turned to 180 degrees
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Connections:
- C2 pad 1: GroundB -> GND
- C3 pad 2: GroundB -> GND
- C4 pad 2: GroundB -> GND
- C5 pad 1: GroundB -> GND
- C6 pad 2: GroundB -> GND
- C7 pad 1: GroundB -> GND
- C8 pad 1: Conn4B -> Conn3B
- C8 pad 2: GroundB -> GND
- D1 pad 2: GroundB -> GND
- D2 pad 1: Net-(D2-Pad1) -> -12V
- D3 pad 2: Net-(D3-Pad2) -> +12V
- J2 pad 1: Net-(D2-Pad1) -> -12V
- J2 pad 10: Net-(D3-Pad2) -> +12V
- J2 pad 2: Net-(D2-Pad1) -> -12V
- J2 pad 3: GroundB -> GND
- J2 pad 4: GroundB -> GND
- J2 pad 5: GroundB -> GND
- J2 pad 6: GroundB -> GND
- J2 pad 7: GroundB -> GND
- J2 pad 8: GroundB -> GND
- J2 pad 9: Net-(D3-Pad2) -> +12V
- J7 pad 1: Conn1B -> GateJackB
- J7 pad 2: GroundB -> Conn1B
- J7 pad 3: Conn3B -> Conn2B
- J7 pad 4: Conn4B -> Switch2B
- J8 pad 1: GateJackB -> Switch1B
- J8 pad 2: OutJackB -> Conn3B
- J8 pad 3: InvOutJackB' -> OutJackB
- J8 pad 4: Switch1B -> InvOutJackB'
- J8 pad 5: Switch2B -> GND
- R1 pad 2: GroundB -> GND
- R12 pad 2: GroundB -> GND
- R3 pad 1: unconnected-(R3-Pad1) -> GND
- R7 pad 2: GroundB -> GND
- U1 pad 8: Conn3B -> Conn2B
- U1 pad 9: Conn3B -> Conn2B
- U2 pad 3: Conn4B -> Conn3B
- U2 pad 4: +12V -> -12V
- U2 pad 8: -12V -> +12V
Routing:
- net -12V: track 0.00 -> 83.9 mm
- net +12V: track 0.00 -> 75.5 mm
- net Switch1B: track 0.00 -> 48.8 mm
- net OutJackB: track 0.00 -> 48.8 mm
- net Conn3B: track 0.00 -> 34.2 mm
- net Net-(R6-Pad1): track 0.00 -> 33.1 mm
- net Conn2B: track 0.00 -> 31.6 mm
- net Net-(R2-Pad1): track 0.00 -> 28.8 mm
- net Switch2B: track 0.00 -> 26.2 mm
- net GateJackB: track 0.00 -> 23.9 mm
- net Net-(C1-Pad1): track 0.00 -> 23.1 mm
- net Net-(R11-Pad2): track 0.00 -> 20.5 mm
- net Conn1B: track 0.00 -> 8.29 mm
- net InvOutJackB': track 0.00 -> 4.34 mm
- added copper zone on B.Cu, net GND
Other:
- board outline added: 20 x 77.7 mm

Commit message: finish traces
Parts:
- moved C8 11.0 mm to (171.9, 107.3)
- moved C5 3.98 mm to (176.1, 106.1)
- moved R10 3.45 mm to (188.0, 110.6)
- moved D1 2.74 mm to (188.1, 96.4)
- moved R12 0.30 mm to (188.2, 128.7)
Connections:
- C2 pad 2: -12V -> -12
- C3 pad 1: +12V -> +12
- C4 pad 1: -12V -> -12
- C5 pad 2: +12V -> +12
- C6 pad 1: -12V -> -12
- C7 pad 2: +12V -> +12
- D2 pad 2: -12V -> -12
- D3 pad 1: +12V -> +12
- R10 pad 1: +12V -> +12
- R2 pad 2: +12V -> +12
- R9 pad 2: +12V -> +12
- U1 pad 11: -12V -> -12
- U1 pad 4: +12V -> +12
- U2 pad 4: -12V -> -12
- U2 pad 8: +12V -> +12
Routing:
- net -12V: track 83.9 -> 6.78 mm
- net -12: track 0.00 -> 77.2 mm
- net +12V: track 75.5 -> 6.91 mm
- net +12: track 0.00 -> 67.3 mm
- net Switch3B: track 0.00 -> 28.3 mm
- net Net-(R10-Pad2): track 0.00 -> 13.7 mm
- net GND: track 0.00 -> 12.6 mm, vias 0 -> 2
- net InvOutJackB': track 4.34 -> 16.7 mm
- net Conn3B: track 34.2 -> 24.3 mm
- net OutJackB: track 48.8 -> 39.2 mm
- net Net-(R11-Pad2): track 20.5 -> 26.9 mm
- net Net-(C1-Pad1): track 23.1 -> 23.9 mm

Commit message: fix connector position
Parts:
- moved J7 7.60 mm to (183.4, 80.0), turned to -90 degrees
Routing:
- net Conn2B: track 31.6 -> 15.8 mm
- net Switch2B: track 26.2 -> 15.9 mm
- net GateJackB: track 23.6 -> 20.9 mm
- net Conn1B: track 8.29 -> 7.58 mm
Changed lines of the file:
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@@
     )
   )
-  (footprint "Connector_PinSocket_2.54mm:PinSocket_1x04_P2.54mm_Vertical" locked (layer "F.Cu")
-    (at 175.768 79.985 90)
+  (footprint "Connector_PinSocket_2.54mm:PinSocket_1x04_P2.54mm_Vertical" (layer "F.Cu")
+    (at 183.368 79.9846 -90)
     (descr "Through hole straight socket strip, 1x04, 2.54mm pitch, single row (from Kicad 4.0.7), script generated")
     (tags "Through hole socket strip THT 1x04 2.54mm single row")
@@
     (property "Sheetname" "")
     (attr through_hole)
-    (fp_text reference "J7" (at 3.1754 3.5052 180) (layer "F.SilkS")
+    (fp_text reference "J7" (at 3.1754 3.5052) (layer "F.SilkS")
       (effects (font (size 1 1) (thickness 0.15)))
     )
@@
     (fp_line (start 0.635 -1.27) (end 1.27 -0.635) (layer "F.Fab") (width 0.1))
     (fp_line (start 1.27 8.89) (end -1.27 8.89) (layer "F.Fab") (width 0.1))
-    (pad "1" thru_hole rect locked (at 0 0 90) (size 1.7 1.7) (drill 1) (layers *.Cu *.Mask)
+    (pad "1" thru_hole rect locked (at 0 0 270) (size 1.7 1.7) (drill 1) (layers *.Cu *.Mask)
       (net 2 "GateJackB") (pinfunction "Pin_1") (pintype "passive"))
-    (pad "2" thru_hole oval locked (at 0 2.54 90) (size 1.7 1.7) (drill 1) (layers *.Cu *.Mask)
+    (pad "2" thru_hole oval locked (at 0 2.54 270) (size 1.7 1.7) (drill 1) (layers *.Cu *.Mask)
       (net 6 "Conn1B") (pinfunction "Pin_2") (pintype "passive"))
-    (pad "3" thru_hole oval locked (at 0 5.08 90) (size 1.7 1.7) (drill 1) (layers *.Cu *.Mask)
+    (pad "3" thru_hole oval locked (at 0 5.08 270) (size 1.7 1.7) (drill 1) (layers *.Cu *.Mask)
       (net 5 "Conn2B") (pinfunction "Pin_3") (pintype "passive"))
-    (pad "4" thru_hole oval locked (at 0 7.62 90) (size 1.7 1.7) (drill 1) (layers *.Cu *.Mask)
+    (pad "4" thru_hole oval locked (at 0 7.62 270) (size 1.7 1.7) (drill 1) (layers *.Cu *.Mask)
       (net 11 "Switch2B") (pinfunction "Pin_4") (pintype "passive"))
     (model "${KICAD6_3DMODEL_DIR}/Connector_PinSocket_2.54mm.3dshapes/PinSocket_1x04_P2.54mm_Vertical.wrl"
@@
   (segment (start 182.6668 96.6266) (end 184.125 96.6266) (width 0.5) (layer "B.Cu") (net 1))
   (segment (start 188.4964 93.38657) (end 188.4964 81.8672) (width 0.5) (layer "B.Cu") (net 1))
-  (segment (start 180.989413 87.212613) (end 181.4934 87.7166) (width 0.5) (layer "B.Cu") (net 2))
-  (segment (start 176.189967 79.985) (end 180.989413 84.784446) (width 0.5) (layer "B.Cu") (net 2))
+  (segment (start 180.998 83.705767) (end 180.998 82.1182) (width 0.5) (layer "B.Cu") (net 2))
+  (segment (start 183.3856 84.6582) (end 181.950433 84.6582) (width 0.5) (layer "B.Cu") (net 2))
+  (segment (start 185.5724 92.6792) (end 187.0764 91.1752) (width 0.5) (layer "B.Cu") (net 2))
+  (segment (start 184.3168 85.5894) (end 183.3856 84.6582) (width 0.5) (layer "B.Cu") (net 2))
+  (segment (start 187.0764 89.97155) (end 184.3168 87.21195) (width 0.5) (layer "B.Cu") (net 2))
+  (segment (start 184.3168 87.21195) (end 184.3168 85.5894) (width 0.5) (layer "B.Cu") (net 2))
   (segment (start 184.638 91.7448) (end 184.5056 91.7448) (width 0.5) (layer "B.Cu") (net 2))
-  (segment (start 185.5724 92.6792) (end 187.0964 91.1552) (width 0.5) (layer "B.Cu") (net 2))
-  (segment (start 175.768 79.985) (end 176.189967 79.985) (width 0.5) (layer "B.Cu") (net 2))
   (segment (start 184.5056 91.7448) (end 184.3074 91.5466) (width 0.5) (layer "B.Cu") (net 2))
   (segment (start 185.5724 92.6792) (end 184.638 91.7448) (width 0.5) (layer "B.Cu") (net 2))
-  (segment (start 186.324167 89.2556) (end 185.1152 89.2556) (width 0.5) (layer "B.Cu") (net 2))
-  (segment (start 181.4934 87.7166) (end 183.5762 87.7166) (width 0.5) (layer "B.Cu") (net 2))
-  (segment (start 180.989413 84.784446) (end 180.989413 87.212613) (width 0.5) (layer "B.Cu") (net 2))
-  (segment (start 187.0964 91.1552) (end 187.0964 90.027833) (width 0.5) (layer "B.Cu") (net 2))
-  (segment (start 187.0964 90.027833) (end 186.324167 89.2556) (width 0.5) (layer "B.Cu") (net 2))
+  (segment (start 187.0764 91.1752) (end 187.0764 89.97155) (width 0.5) (layer "B.Cu") (net 2))
+  (segment (start 180.998 82.1182) (end 183.1316 79.9846) (width 0.5) (layer "B.Cu") (net 2))
   (segment (start 184.3074 91.5466) (end 182.6668 91.5466) (width 0.5) (layer "B.Cu") (net 2))
-  (segment (start 183.5762 87.7166) (end 185.1152 89.2556) (width 0.5) (layer "B.Cu") (net 2))
+  (segment (start 181.950433 84.6582) (end 180.998 83.705767) (width 0.5) (layer "B.Cu") (net 2))
   (segment (start 174.306112 60.085088) (end 171.8564 62.5348) (width 0.5) (layer "B.Cu") (net 3))
   (segment (start 174.306112 59.309) (end 174.306112 60.085088) (width 0.5) (layer "B.Cu") (net 3))
@@
   (segment (start 184.466112 59.309) (end 184.466112 59.853712) (width 0.5) (layer "B.Cu") (net 4))
   (segment (start 184.466112 56.769) (end 184.466112 59.309) (width 0.5) (layer "B.Cu") (net 4))
-  (segment (start 180.848 79.985) (end 182.148 81.285) (width 0.5) (layer "B.Cu") (net 5))
-  (segment (start 182.148 81.285) (end 184.0942 81.285) (width 0.5) (layer "B.Cu") (net 5))
-  (segment (start 173.3346 86.4666) (end 175.0468 86.4666) (width 0.5) (layer "B.Cu") (net 5))
-  (segment (start 174.0408 77.6224) (end 173.0756 78.5876) (width 0.5) (layer "B.Cu") (net 5))
-  (segment (start 172.5676 85.6996) (end 173.3346 86.4666) (width 0.5) (layer "B.Cu") (net 5))
-  (segment (start 184.0942 81.285) (end 184.8612 80.518) (width 0.5) (layer "B.Cu") (net 5))
+  (segment (start 173.7844 79.873322) (end 173.7844 80.72185) (width 0.5) (layer "B.Cu") (net 5))
+  (segment (start 172.802 84.2218) (end 175.0468 86.4666) (width 0.5) (layer "B.Cu") (net 5))
+  (segment (start 174.973122 78.6846) (end 173.7844 79.873322) (width 0.5) (layer "B.Cu") (net 5))
+  (segment (start 176.7516 78.6846) (end 174.973122 78.6846) (width 0.5) (layer "B.Cu") (net 5))
+  (segment (start 178.0516 79.9846) (end 176.7516 78.6846) (width 0.5) (layer "B.Cu") (net 5))
   (segment (start 175.0468 89.0066) (end 175.0468 86.4666) (width 0.5) (layer "B.Cu") (net 5))
-  (segment (start 173.0756 80.9752) (end 172.5676 81.4832) (width 0.5) (layer "B.Cu") (net 5))
-  (segment (start 183.0832 77.6224) (end 174.0408 77.6224) (width 0.5) (layer "B.Cu") (net 5))
-  (segment (start 173.0756 78.5876) (end 173.0756 80.9752) (width 0.5) (layer "B.Cu") (net 5))
-  (segment (start 184.8612 80.518) (end 184.8612 79.4004) (width 0.5) (layer "B.Cu") (net 5))
-  (segment (start 184.8612 79.4004) (end 183.0832 77.6224) (width 0.5) (layer "B.Cu") (net 5))
-  (segment (start 172.5676 81.4832) (end 172.5676 85.6996) (width 0.5) (layer "B.Cu") (net 5))
-  (segment (start 178.308 81.113083) (end 182.6668 85.471883) (width 0.5) (layer "B.Cu") (net 6))
-  (segment (start 182.6668 85.471883) (end 182.6668 86.4666) (width 0.5) (layer "B.Cu") (net 6))
-  (segment (start 178.308 79.985) (end 178.308 81.113083) (width 0.5) (layer "B.Cu") (net 6))
+  (segment (start 173.7844 80.72185) (end 172.802 81.70425) (width 0.5) (layer "B.Cu") (net 5))
+  (segment (start 172.802 81.70425) (end 172.802 84.2218) (width 0.5) (layer "B.Cu") (net 5))
+  (segment (start 180.298 84.0978) (end 182.6668 86.4666) (width 0.5) (layer "B.Cu") (net 6))
+  (segment (start 180.298 80.2782) (end 180.298 84.0978) (width 0.5) (layer "B.Cu") (net 6))
+  (segment (start 180.5916 79.9846) (end 180.298 80.2782) (width 0.5) (layer "B.Cu") (net 6))
   (segment (start 175.783 122.29525) (end 176.416866 122.29525) (width 0.5) (layer "B.Cu") (net 7))
   (segment (start 177.960517 115.6716) (end 177.3428 115.6716) (width 0.5) (layer "B.Cu") (net 7))
@@
   (segment (start 173.243 121.701801) (end 175.457523 119.487278) (width 0.5) (layer "B.Cu") (net 10))
   (segment (start 178.234889 119.487278) (end 178.9928 118.729367) (width 0.5) (layer "B.Cu") (net 10))
-  (segment (start 176.3776 85.1916) (end 174.5996 85.1916) (width 0.5) (layer "B.Cu") (net 11))
-  (segment (start 174.483602 78.3844) (end 181.7874 78.3844) (width 0.5) (layer "B.Cu") (net 11))
-  (segment (start 173.482 84.074) (end 173.482 81.55875) (width 0.5) (layer "B.Cu") (net 11))
-  (segment (start 174.5996 85.1916) (end 173.482 84.074) (width 0.5) (layer "B.Cu") (net 11))
-  (segment (start 175.0468 91.5466) (end 176.7332 89.8602) (width 0.5) (layer "B.Cu") (net 11))
-  (segment (start 181.7874 78.3844) (end 183.388 79.985) (width 0.5) (layer "B.Cu") (net 11))
-  (segment (start 176.7332 89.8602) (end 176.7332 85.5472) (width 0.5) (layer "B.Cu") (net 11))
-  (segment (start 176.7332 85.5472) (end 176.3776 85.1916) (width 0.5) (layer "B.Cu") (net 11))
-  (segment (start 173.8884 78.979602) (end 174.483602 78.3844) (width 0.5) (layer "B.Cu") (net 11))
-  (segment (start 173.8884 81.15235) (end 173.8884 78.979602) (width 0.5) (layer "B.Cu") (net 11))
-  (segment (start 173.482 81.55875) (end 173.8884 81.15235) (width 0.5) (layer "B.Cu") (net 11))
+  (segment (start 177.0492 85.3322) (end 176.3244 84.6074) (width 0.5) (layer "B.Cu") (net 11))
+  (segment (start 175.0468 91.5466) (end 177.0492 89.5442) (width 0.5) (layer "B.Cu") (net 11))
+  (segment (start 176.3244 84.6074) (end 174.279633 84.6074) (width 0.5) (layer "B.Cu") (net 11))
+  (segment (start 173.502 81.9942) (end 175.5116 79.9846) (width 0.5) (layer "B.Cu") (net 11))
+  (segment (start 173.502 83.829767) (end 173.502 81.9942) (width 0.5) (layer "B.Cu") (net 11))
+  (segment (start 174.279633 84.6074) (end 173.502 83.829767) (width 0.5) (layer "B.Cu") (net 11))
+  (segment (start 177.0492 89.5442) (end 177.0492 85.3322) (width 0.5) (layer "B.Cu") (net 11))
   (segment (start 185.943 122.29525) (end 185.7705 122.29525) (width 0.5) (layer "B.Cu") (net 12))
   (segment (start 182.5864 119.11115) (end 182.5864 115.762) (width 0.5) (layer "B.Cu") (net 12))
