File: ASREnvelope/ASREnvelope_control/ASREnvelope_control.kicad_pcb (KiCad board)
At the start: 2 copper layers, 20 x 100 mm, 19 parts, among them J1 GATE, J3 OUT, J4 INV OUT, J5 Conn_01x06_Male, J6 Conn_01x04_Male, SW1 SW_SPDT

Commit message: fix errors
Parts:
- moved D5 25.2 mm to (155.3, 88.2), turned to 180 degrees
- moved D7 15.2 mm to (158.7, 53.2)
- moved R8 14.1 mm to (147.3, 65.8), turned to 0 degrees
- moved D4 0.38 mm to (158.4, 107.1)
Connections:
- R4 pad 1: Switch3A -> Net-(D4-Pad1)
Routing:
- net Net-(D5-Pad1): track 75.5 -> 21.6 mm
- net Conn1A: track 25.4 -> 6.10 mm
- net Net-(D7-Pad2): track 34.0 -> 15.3 mm
- net Net-(D8-Pad2): track 32.7 -> 20.6 mm
- net Net-(D4-Pad1): track 4.32 -> 15.8 mm
- net Conn2A: track 30.4 -> 40.3 mm
- net Conn3A: track 100.2 -> 94.2 mm
- net Net-(D7-Pad1): track 7.03 -> 12.5 mm
- net Switch2A: track 46.3 -> 42.9 mm
- net Switch3A: track 32.0 -> 29.2 mm
- net GateJackA: track 41.7 -> 40.9 mm
